Commit message: added readme, requirements.txt, fixes made to get project running again

File: src/norby_webots_drivers/urdf/TurtleBot3Burger.urdf (robot description, URDF)
Before this commit: robot TurtleBot3Burger, 14 links, 13 joints
Links:
- added link gps_link
- added link imu_link
Joints:
- added joint base_link_gps_joint: type fixed, parent base_link, child gps_link, origin xyz=-0.03 0 0.153 rpy=0 0 0
- added joint base_link_imu_joint: type fixed, parent base_link, child imu_link, origin xyz=-0.032 0 0.078 rpy=0 0 0
